Commit message: 1. update the urdf model 2. update the parameters

File: source/rl_training/data/Robots/deeprobotics/lite3_description/urdf/lite3.urdf (robot description, URDF)
Before this commit: robot Lite3, 17 links, 16 joints
Links:
- link FL_FOOT: geometry collision sphere radius=0.022
- link FL_HIP: geometry collision cylinder length=0.15 radius=0.04; visual mesh filename=../meshes/hip.STL scale=1 1 1
- link FL_SHANK: geometry collision cylinder length=0.10 radius=0.015; collision cylinder length=0.12 radius=0.015
- link FL_THIGH: geometry collision box size=0.04 0.045 0.2; visual mesh filename=../meshes/thigh.STL
- link FR_FOOT: geometry collision sphere radius=0.022
- link FR_HIP: geometry collision cylinder length=0.15 radius=0.04; visual mesh filename=../meshes/hip.STL scale=1 -1 1
- link FR_SHANK: geometry collision cylinder length=0.10 radius=0.015; collision cylinder length=0.12 radius=0.015
- link FR_THIGH: geometry collision box size=0.04 0.045 0.2; visual mesh filename=../meshes/thigh.STL scale=1 -1 1
- link HL_FOOT: geometry collision sphere radius=0.022
- link HL_HIP: geometry collision cylinder length=0.15 radius=0.04; visual mesh filename=../meshes/hip.STL scale=-1 1 1
- link HL_SHANK: geometry collision cylinder length=0.10 radius=0.015; collision cylinder length=0.12 radius=0.015
- link HL_THIGH: geometry collision box size=0.04 0.045 0.2; visual mesh filename=../meshes/thigh.STL
- link HR_FOOT: geometry collision sphere radius=0.022
- link HR_HIP: geometry collision cylinder length=0.15 radius=0.04; visual mesh filename=../meshes/hip.STL scale=-1 -1 1
- link HR_SHANK: geometry collision cylinder length=0.10 radius=0.015; collision cylinder length=0.12 radius=0.015
- link HR_THIGH: geometry collision box size=0.04 0.045 0.2; visual mesh filename=../meshes/thigh.STL scale=1 -1 1
Joints:
- joint FL_HipX_joint: origin xyz=0.1745 0.062 0 rpy=0 0 0 -> xyz=0.1745 0.062 0
- joint FL_HipY_joint: origin xyz=0 0.09735 0 rpy=0 0 0 -> xyz=0 0.09735 0
- joint FL_Knee_joint: origin xyz=0 0 -0.20 rpy=0 0 0 -> xyz=0 0 -0.20
- joint FR_HipX_joint: origin xyz=0.1745 -0.062 0 rpy=0 0 0 -> xyz=0.1745 -0.062 0
- joint FR_HipY_joint: origin xyz=0 -0.09735 0 rpy=0 0 0 -> xyz=0 -0.09735 0
- joint FR_Knee_joint: origin xyz=0 0 -0.20 rpy=0 0 0 -> xyz=0 0 -0.20
- joint HL_HipX_joint: origin xyz=-0.1745 0.062 0 rpy=0 0 0 -> xyz=-0.1745 0.062 0
- joint HL_HipY_joint: origin xyz=0 0.09735 0 rpy=0 0 0 -> xyz=0 0.09735 0
- joint HL_Knee_joint: origin xyz=0 0 -0.20 rpy=0 0 0 -> xyz=0 0 -0.20
- joint HR_HipX_joint: origin xyz=-0.1745 -0.062 0 rpy=0 0 0 -> xyz=-0.1745 -0.062 0
- joint HR_HipY_joint: origin xyz=0 -0.09735 0 rpy=0 0 0 -> xyz=0 -0.09735 0
- joint HR_Knee_joint: origin xyz=0 0 -0.20 rpy=0 0 0 -> xyz=0 0 -0.20
